Commit message: remove unnecessary collision meshes

File: awd/data/assets/go_bdx/go_bdx.urdf (robot description, URDF)
Before this commit: robot bdx, 21 links, 20 joints
Links:
- link head_body_pitch: geometry visual mesh filename=meshes/head_body_pitch.stl scale=0.001 0.001 0.001
- link head_body_yaw: geometry visual mesh filename=meshes/head_body_yaw.stl scale=0.001 0.001 0.001
- link left_hip: geometry visual mesh filename=meshes/left_hip.stl scale=0.001 0.001 0.001
- link left_hip_rotation: geometry visual mesh filename=meshes/left_hip_rotation.stl scale=0.001 0.001 0.001
- link left_thigh: geometry visual mesh filename=meshes/left_thigh.stl scale=0.001 0.001 0.001
- link neck: geometry visual mesh filename=meshes/neck.stl scale=0.001 0.001 0.001
- link right_hip: geometry visual mesh filename=meshes/right_hip.stl scale=0.001 0.001 0.001
- link right_hip_rotation: geometry visual mesh filename=meshes/right_hip_rotation.stl scale=0.001 0.001 0.001
- link right_thigh: geometry visual mesh filename=meshes/right_thigh.stl scale=0.001 0.001 0.001
