Commit message: add mini2 bdx abd fix mini1 bdx urdf

File: awd/data/assets/mini_bdx/urdf/bdx.urdf (robot description, URDF)
Before this commit: robot bdx, 20 links, 19 joints
Links:
- link body_module: geometry collision mesh filename=../meshes/39281023.prt.stl; collision mesh filename=../meshes/bms.stl
- link double_u_module: geometry collision mesh filename=../meshes/dc15_a01_horn_dummy.stl; collision mesh filename=../meshes/dc15_a01_horn_dummy.stl
- link double_u_module_2: geometry collision mesh filename=../meshes/dc15_a01_horn_dummy.stl; collision mesh filename=../meshes/dc15_a01_horn_dummy.stl
- link foot_module: geometry collision mesh filename=../meshes/dc15_a01_horn_dummy.stl; collision mesh filename=../meshes/dc15_a01_horn_idle2_dummy.stl
- link foot_module_2: geometry collision mesh filename=../meshes/dc15_a01_horn_dummy.stl; collision mesh filename=../meshes/dc15_a01_horn_idle2_dummy.stl
- link head_assembly: geometry collision mesh filename=../meshes/antenna_motor_holder.stl; collision mesh filename=../meshes/antenna_motor_holder.stl
- link head_link: geometry collision mesh filename=../meshes/axis_to_axis.stl; collision mesh filename=../meshes/axis_to_axis.stl
- link head_pitch_yaw: geometry collision mesh filename=../meshes/dc15_a01_case_b_dummy.stl; collision mesh filename=../meshes/dc15_a01_case_b_dummy.stl
- link left_antenna_assembly: geometry collision mesh filename=../meshes/antenna.stl; collision mesh filename=../meshes/antenna_holder_left.stl
- link left_hip_pitch_roll_module: geometry collision mesh filename=../meshes/dc15_a01_case_b_dummy.stl; collision mesh filename=../meshes/dc15_a01_case_b_dummy.stl
- link leg_module: geometry collision mesh filename=../meshes/block_to_axis.stl; collision mesh filename=../meshes/block_to_axis.stl
- link leg_module_2: geometry collision mesh filename=../meshes/block_to_axis.stl; collision mesh filename=../meshes/block_to_axis.stl
- link leg_module_3: geometry collision mesh filename=../meshes/block_to_axis.stl; collision mesh filename=../meshes/block_to_axis.stl
- link leg_module_4: geometry collision mesh filename=../meshes/block_to_axis.stl; collision mesh filename=../meshes/block_to_axis.stl
- link right_antenna_assembly: geometry collision mesh filename=../meshes/antenna.stl; collision mesh filename=../meshes/antenna_holder_right.stl
- link right_hip_pitch_roll_module: geometry collision mesh filename=../meshes/dc15_a01_case_b_dummy.stl; collision mesh filename=../meshes/dc15_a01_case_b_dummy.stl
Joints:
- joint head_pitch: limit lower=-0.69813170079773179122 upper=0.69813170079773179122 effort=0.52 velocity=10.7 -> lower=-0.69813170079773179122 upper=0.69813170079773179122 effort=0.4 velocity=10.7
- joint head_yaw: limit lower=-2.0943951023931952626 upper=2.0943951023931952626 effort=0.52 velocity=10.7 -> lower=-2.0943951023931952626 upper=2.0943951023931952626 effort=0.4 velocity=10.7
- joint left_ankle: limit lower=-1.570796326794896558 upper=1.570796326794896558 effort=0.93 velocity=8.48 -> lower=-1.570796326794896558 upper=1.570796326794896558 effort=0.80 velocity=8.48
- joint left_hip_pitch: limit lower=-0.52359877559829881566 upper=1.570796326794896558 effort=0.93 velocity=8.48 -> lower=-0.52359877559829881566 upper=1.570796326794896558 effort=0.80 velocity=8.48
- joint left_hip_roll: limit lower=-1.570796326794896558 upper=0.43633231299858238339 effort=0.93 velocity=8.48 -> lower=-1.570796326794896558 upper=0.43633231299858238339 effort=0.80 velocity=8.48
- joint left_hip_yaw: limit lower=-0.69813170079773179122 upper=0.69813170079773179122 effort=0.93 velocity=8.48 -> lower=-0.69813170079773179122 upper=0.69813170079773179122 effort=0.80 velocity=8.48
- joint left_knee: limit lower=-2.0943951023931952626 upper=2.0943951023931952626 effort=0.93 velocity=8.48 -> lower=-2.0943951023931952626 upper=2.0943951023931952626 effort=0.80 velocity=8.48
- joint neck_pitch: limit lower=-1.3089969389957472057 upper=0.1745329251994329478 effort=0.52 velocity=10.7 -> lower=-1.3089969389957472057 upper=0.1745329251994329478 effort=0.4 velocity=10.7
- joint right_ankle: limit lower=-1.570796326794896558 upper=1.570796326794896558 effort=0.93 velocity=8.48 -> lower=-1.570796326794896558 upper=1.570796326794896558 effort=0.80 velocity=8.48
- joint right_hip_pitch: limit lower=-0.52359877559829881566 upper=1.570796326794896558 effort=0.93 velocity=8.48 -> lower=-0.52359877559829881566 upper=1.570796326794896558 effort=0.80 velocity=8.48
- joint right_hip_roll: limit lower=-1.570796326794896558 upper=0.43633231299858238339 effort=0.93 velocity=8.48 -> lower=-1.570796326794896558 upper=0.43633231299858238339 effort=0.80 velocity=8.48
- joint right_hip_yaw: limit lower=-0.69813170079773179122 upper=0.69813170079773179122 effort=0.93 velocity=8.48 -> lower=-0.69813170079773179122 upper=0.69813170079773179122 effort=0.80 velocity=8.48
- joint right_knee: limit lower=-2.0943951023931952626 upper=2.0943951023931952626 effort=0.93 velocity=8.48 -> lower=-2.0943951023931952626 upper=2.0943951023931952626 effort=0.80 velocity=8.48
