Commit message: new urdf

File: awd/data/assets/mini2_bdx/mini2_bdx.urdf (robot description, URDF)
Before this commit: robot onshape, 18 links, 17 joints
Links:
- removed link head_pitch_assembly
- removed link neck_assembly
- added link head_pitch_to_yaw, mass 0.016937787992335997383; collision mesh filename=./head_pitch_to_yaw.stl; visual mesh filename=./head_pitch_to_yaw.stl
- added link left_antenna_holder, mass 0.0042162890957708797426; collision mesh filename=./antenna.stl; collision mesh filename=./left_antenna_holder.stl
- added link neck_pitch_assembly, mass 0.066180000000000058225; collision mesh filename=./neck_left_sheet.stl; collision mesh filename=./neck_right_sheet.stl
- added link neck_yaw_assembly, mass 0.09180988857925044544; collision mesh filename=./head_yaw_to_roll.stl; visual mesh filename=./head_yaw_to_roll.stl
- added link right_antenna_holder, mass 0.004216286984950681424; collision mesh filename=./antenna.stl; collision mesh filename=./right_antenna_holder.stl
- link foot_assembly: mass 0.056240000000000012204 -> 0.075240000000000001323; geometry collision mesh filename=./foot_bottom_pla.stl; collision mesh filename=./foot_bottom_tpu.stl
- link foot_assembly_2: mass 0.056240000000000012204 -> 0.075240000000000001323; geometry collision mesh filename=./foot_bottom_pla.stl; collision mesh filename=./foot_bottom_tpu.stl
- link head_assembly: mass 0.22929000000000004933 -> 0.35258298534369564292; geometry collision mesh filename=./board.stl; collision mesh filename=./head.stl
- link hip_roll_assembly: mass 0.066480000000000011307 -> 0.06648000000000005294; geometry collision mesh filename=./roll_motor_bottom.stl; collision mesh filename=./roll_motor_top.stl
- link hip_roll_assembly_2: mass 0.066480000000000011307 -> 0.06648000000000005294; geometry collision mesh filename=./roll_motor_bottom.stl; collision mesh filename=./roll_motor_top.stl
- link knee_and_ankle_assembly: mass 0.12406999999999994422 -> 0.12407000000000001361; geometry collision mesh filename=./left_cache.stl; collision mesh filename=./left_knee_to_ankle_left_sheet.stl
- link knee_and_ankle_assembly_2: mass 0.072590000000000015623 -> 0.072590000000000057256; geometry collision mesh filename=./left_knee_to_ankle_left_sheet.stl; collision mesh filename=./left_knee_to_ankle_right_sheet.stl
- link knee_and_ankle_assembly_3: mass 0.12407000000000002748 -> 0.12407000000000001361; geometry collision mesh filename=./left_knee_to_ankle_left_sheet.stl; collision mesh filename=./left_knee_to_ankle_right_sheet.stl
- link knee_and_ankle_assembly_4: mass 0.072590000000000015623 -> 0.072590000000000057256; geometry collision mesh filename=./left_knee_to_ankle_left_sheet.stl; collision mesh filename=./left_knee_to_ankle_right_sheet.stl
- link left_roll_to_pitch_assembly: mass 0.075160000000000018461 -> 0.075160000000000060094; geometry collision mesh filename=./left_roll_to_pitch.stl; visual mesh filename=./left_roll_to_pitch.stl
- link right_roll_to_pitch_assembly: mass 0.075160000000000018461 -> 0.075160000000000060094; geometry collision mesh filename=./right_roll_to_pitch.stl; visual mesh filename=./right_roll_to_pitch.stl
- link trunk_assembly: mass 0.55922072109020470876 -> 0.69852641931996084512; geometry collision mesh filename=./battery_pack_lid.stl; collision mesh filename=./bms.stl
Joints:
- added joint head_roll: type revolute, parent neck_yaw_assembly, child head_assembly, origin xyz=0.040950000000000097433 -1.7527483370943786056e-16 -0.019149999999999778311 rpy=-7.3227915058204641542e-14 -1.570796326794896336 0, axis 0 0 1, limit lower=-0.52359877559829881566 upper=0.52359877559829881566 effort=1 velocity=20
- added joint left_antenna: type revolute, parent head_assembly, child left_antenna_holder, origin xyz=0.00070406945503534434927 0.060662837687359784378 0.11643485329544212004 rpy=-3.1415926535896234739 1.3045791727887248168 1.3234423712232488146, axis 0 0 1, limit lower=-1.570796326794896558 upper=1.570796326794896558 effort=1 velocity=20
- added joint right_antenna: type revolute, parent head_assembly, child right_antenna_holder, origin xyz=0.00070406945503534434927 -0.06066283768735826476 0.11643485329544212004 rpy=3.1415926535896230298 1.3045791727887245948 -1.3234423712232490367, axis 0 0 1, limit lower=-1.570796326794896558 upper=1.570796326794896558 effort=1 velocity=20
- joint head_frame: origin xyz=4.1633363423443370266e-17 0 -0.01249999999999990008 rpy=-3.1415926535897797933 4.3716373664754018489e-18 7.4988647406086779923e-30 -> xyz=0.04245000000000057061 7.4178402136026999614e-16 0.035949999999999988909 rpy=2.2204460492701854731e-16 1.570796326794896336 0
- joint head_pitch: child head_pitch_assembly -> head_pitch_to_yaw; limit lower=-1.570796326794896558 upper=1.570796326794896558 effort=1 velocity=20 -> lower=-0.785398163397448279 upper=0.785398163397448279 effort=1 velocity=20; origin xyz=1.0408340855860842566e-16 0.066000000000000391687 -3.4694469519536141888e-18 rpy=-1.0915849447069766081e-16 -7.3845547632106068786e-17 -1.0417200973690603325e-16 -> xyz=8.6736173798840354721e-19 0.066000000000000016986 -3.4694469519536141888e-18 rpy=-1.4406834481465239151e-16 -1.1423136877781657605e-16 1.1213426021061680001e-13; parent neck_assembly -> neck_pitch_assembly
- joint head_yaw: child head_assembly -> neck_yaw_assembly; limit lower=-2.9670597283903603625 upper=2.9670597283903603625 effort=1 velocity=20 -> lower=-2.7925268031909271649 upper=2.7925268031909271649 effort=1 velocity=20; origin xyz=-2.0816681711721685133e-17 0.056900000000000033884 0.019049999999999952388 rpy=1.5707963267948958919 -2.9140480977164958126e-15 -8.9523033089878119206e-15 -> xyz=-1.6913553890773869171e-17 0.056999999999999939604 0.019050000000000014838 rpy=-1.570796326794896558 7.3522809646371816617e-14 6.1232339957365034931e-17; parent head_pitch_assembly -> head_pitch_to_yaw
- joint left_ankle: origin xyz=0 -0.07865000000000006708 9.9999999999988986588e-05 rpy=-5.5077724532749743024e-16 9.2653469445928301633e-16 3.2402024558001311503e-14 -> xyz=-3.4694469519536141888e-17 -0.078650000000000178102 9.99999999999751088e-05 rpy=-2.6413756774523519415e-16 1.2220841311108591179e-26 2.7755576181993178136e-17
- joint left_foot_frame: origin xyz=0 -0.036724999999999979883 0.019049999999999983613 rpy=-1.570796326794896558 -3.4146152368508307717e-19 -1.8519077370852487142e-17 -> xyz=0.00049999999999996574962 -0.036224999999999729638 0.01955000000000034488 rpy=-1.570796326794896558 4.8789097742003279458e-18 8.5828066488045564267e-28
- joint left_hip_pitch: limit lower=-1.570796326794896558 upper=0.52359877559829881566 effort=1 velocity=20 -> lower=-1.2217304763960306069 upper=0.52359877559829881566 effort=1 velocity=20; origin xyz=0.074149999999998272848 1.249000902703301108e-15 0.035109999999998510456 rpy=3.1415926535897926719 1.5707963267948574781 0 -> xyz=0.074149999999999799405 1.3959102970750869588e-18 0.035109999999999912113 rpy=3.141592653589793116 1.5707963267948952257 0
- joint left_hip_roll: origin xyz=0.019050000000002648148 1.9602375278537920167e-15 -0.046015000000004538383 rpy=-1.5707963267950215691 1.6937530152664249305e-13 1.5707963267952902431 -> xyz=0.019050000000003241424 2.0469737016526323714e-15 -0.046015000000000895464 rpy=-1.5707963267949442976 1.0251581517556108667e-13 1.5707963267946023489
- joint left_hip_yaw: origin xyz=-0.056394334796673495358 0.028602766445326346934 0.024395090932709764808 rpy=-6.2403804745132919901e-14 0.021825623709755430368 1.3218914061185209833e-13 -> xyz=-0.019000000000000290962 0.035000000000001273148 0.045940938812378845357 rpy=-2.0757017677015319346e-16 -2.1982415887547258194e-14 -7.6136910267405882653e-27
- joint left_knee: origin xyz=-9.7144514654701197287e-17 -0.078649999999999734013 9.9999999999961231012e-05 rpy=7.358361518165846965e-16 5.0845139115396107043e-16 -7.1846367703695162136e-14 -> xyz=1.3877787807814456755e-17 -0.078650000000000011569 9.9999999999961231012e-05 rpy=-2.6413756781799972404e-16 -2.7339812777890022088e-26 0
- joint neck_pitch: child neck_assembly -> neck_pitch_assembly; origin xyz=-0.035437537550831413324 0.012752766445331959258 0.068008119366846808695 rpy=1.5707963267948341635 0.021825623709755184038 1.3218913913091132832e-13 -> xyz=0.00099999999999896352354 0.019150000000000326483 0.090000938812376238274 rpy=1.570796326794896558 8.9928064994637667153e-14 6.1232449686014378908e-17
- joint right_ankle: origin xyz=-2.7755575615628913511e-17 -0.078650000000000080957 9.9999999999961231012e-05 rpy=-2.6194324489465746712e-16 2.8316471284964215798e-29 9.5878895885319479181e-14 -> xyz=-6.9388939039072283776e-18 -0.078650000000000039324 9.9999999999961231012e-05 rpy=-2.6413756984180028828e-16 -6.9382288127881716121e-25 -5.1722034616178551878e-17
- joint right_foot_frame: origin xyz=-1.3877787807814456755e-17 -0.036724999999999979883 0.019049999999999969735 rpy=-1.570796326794896558 -4.7247190275601867229e-17 6.0085748048618062173e-16 -> xyz=0.0005000000000002155498 -0.036224999999999840661 0.019550000000000664069 rpy=-1.570796326794896558 9.1691846176123393012e-16 1.3322725304659061714e-15
- joint right_hip_pitch: limit lower=-0.52359877559829881566 upper=1.570796326794896558 effort=1 velocity=20 -> lower=-0.52359877559829881566 upper=1.2217304763960306069 effort=1 velocity=20; origin xyz=-0.074149999999999993694 -2.0816681711721685133e-17 0.035110000000000009257 rpy=-2.1823850769468260177e-17 1.5707963267948927832 0 -> xyz=-0.074149999999999799405 3.1868767607495795957e-16 0.035110000000000016196 rpy=-2.3836094894413110414e-24 1.570796326794896336 0
- joint right_hip_roll: origin xyz=0.019050000000005999634 2.9060087669563472446e-14 -0.046014999999998154601 rpy=-1.570796326794797082 -7.3141829490872532251e-14 1.5707963267946682961 -> xyz=0.019050000000008261714 3.78516662458139308e-14 -0.046015000000003032643 rpy=-1.5707963267947879782 -8.4491074221037422062e-14 1.5707963267945974639
- joint right_hip_yaw: origin xyz=-0.056394334796664107035 -0.041397233554676490797 0.024395090932713945492 rpy=-5.7479562369434986172e-14 0.021825623709755558738 3.5607454337323585543e-13 -> xyz=-0.018999999999998431338 -0.03500000000000151601 0.045940938812377415945 rpy=-4.6224992538811313716e-16 -2.2037927038832600325e-14 -1.6653345370219725828e-16
- joint right_knee: origin xyz=-1.360023205165816762e-15 0.07864999999999899849 0.036999999999998534062 rpy=3.141592653589793116 -5.3042305426499207572e-15 1.0017539295583627067e-13 -> xyz=-6.9388939039072283776e-18 0.078649999999999414824 0.036999999999999658162 rpy=3.141592653589793116 -2.0819102970830263503e-24 5.0289882707839502595e-30
- joint trunk_frame: origin xyz=-0.060471084556686989508 -0.0063972335546741820184 0.066744147727335195741 rpy=-6.3086333636868837384e-14 0.021825623709755163221 1.3209498708375492755e-13 -> xyz=-0.024000000000000760308 -2.4112656316077618612e-16 0.088190938812376745704 rpy=-1.4062102177136726269e-16 -9.4252837597218562265e-17 7.8061435390716270015e-33

Commit message: mini2

File: awd/data/assets/mini2_bdx/mini2_bdx.urdf (robot description, URDF)
Before this commit: robot onshape, 21 links, 20 joints
Joints:
- joint head_pitch: limit lower=-0.785398163397448279 upper=0.785398163397448279 effort=1 velocity=20 -> lower=-0.785398163397448279 upper=0.785398163397448279 effort=20 velocity=200
- joint head_roll: limit lower=-0.52359877559829881566 upper=0.52359877559829881566 effort=1 velocity=20 -> lower=-0.52359877559829881566 upper=0.52359877559829881566 effort=20 velocity=200
- joint head_yaw: limit lower=-2.7925268031909271649 upper=2.7925268031909271649 effort=1 velocity=20 -> lower=-2.7925268031909271649 upper=2.7925268031909271649 effort=20 velocity=200
- joint left_ankle: limit lower=-1.570796326794896558 upper=1.570796326794896558 effort=1 velocity=20 -> lower=-1.570796326794896558 upper=1.570796326794896558 effort=20 velocity=200
- joint left_antenna: limit lower=-1.570796326794896558 upper=1.570796326794896558 effort=1 velocity=20 -> lower=-1.570796326794896558 upper=1.570796326794896558 effort=20 velocity=200
- joint left_hip_pitch: limit lower=-1.2217304763960306069 upper=0.52359877559829881566 effort=1 velocity=20 -> lower=-1.2217304763960306069 upper=0.52359877559829881566 effort=20 velocity=200
- joint left_hip_roll: limit lower=-0.43633231299858238339 upper=0.43633231299858238339 effort=1 velocity=20 -> lower=-0.43633231299858238339 upper=0.43633231299858238339 effort=20 velocity=200
- joint left_hip_yaw: limit lower=-0.52359877559829881566 upper=0.52359877559829881566 effort=1 velocity=20 -> lower=-0.52359877559829881566 upper=0.52359877559829881566 effort=20 velocity=200
- joint left_knee: limit lower=-1.570796326794896558 upper=1.570796326794896558 effort=1 velocity=20 -> lower=-1.570796326794896558 upper=1.570796326794896558 effort=20 velocity=200
- joint neck_pitch: limit lower=-0.34906585039886589561 upper=1.1344640137963142301 effort=1 velocity=20 -> lower=-0.34906585039886589561 upper=1.1344640137963142301 effort=20 velocity=200
- joint right_ankle: limit lower=-1.570796326794896558 upper=1.570796326794896558 effort=1 velocity=20 -> lower=-1.570796326794896558 upper=1.570796326794896558 effort=20 velocity=200
- joint right_antenna: limit lower=-1.570796326794896558 upper=1.570796326794896558 effort=1 velocity=20 -> lower=-1.570796326794896558 upper=1.570796326794896558 effort=20 velocity=200
- joint right_hip_pitch: limit lower=-0.52359877559829881566 upper=1.2217304763960306069 effort=1 velocity=20 -> lower=-0.52359877559829881566 upper=1.2217304763960306069 effort=20 velocity=200
- joint right_hip_roll: limit lower=-0.43633231299858238339 upper=0.43633231299858238339 effort=1 velocity=20 -> lower=-0.43633231299858238339 upper=0.43633231299858238339 effort=20 velocity=200
- joint right_hip_yaw: limit lower=-0.52359877559829881566 upper=0.52359877559829881566 effort=1 velocity=20 -> lower=-0.52359877559829881566 upper=0.52359877559829881566 effort=20 velocity=200
- joint right_knee: limit lower=-1.570796326794896558 upper=1.570796326794896558 effort=1 velocity=20 -> lower=-1.570796326794896558 upper=1.570796326794896558 effort=20 velocity=200

Commit message: stuff

File: awd/data/assets/mini2_bdx/mini2_bdx.urdf (robot description, URDF)
Before this commit: robot onshape, 21 links, 20 joints
Joints:
- joint left_hip_pitch: limit lower=-1.2217304763960306069 upper=0.52359877559829881566 effort=20 velocity=200 -> lower=-1.570796326794896558 upper=0.72359877559829881566 effort=20 velocity=200
- joint right_hip_pitch: limit lower=-0.52359877559829881566 upper=1.2217304763960306069 effort=20 velocity=200 -> lower=-0.72359877559829881566 upper=1.5707304763960306069 effort=20 velocity=200
