Commit message: update urdf

File: awd/data/assets/mini2_bdx/mini2_bdx.urdf (robot description, URDF)
Before this commit: robot onshape, 21 links, 20 joints
Links:
- link foot_assembly: mass 0.075240000000000001323 -> 0.075240000000000015201
- link foot_assembly_2: mass 0.075240000000000001323 -> 0.075240000000000015201
- link head_assembly: mass 0.35258298534369564292 -> 0.35258298534369525434; geometry collision mesh filename=./board.stl; collision mesh filename=./drive_palonier.stl
- link head_pitch_to_yaw: mass 0.016937787992335997383 -> 0.016937787992336000853
- link hip_roll_assembly: mass 0.06648000000000005294 -> 0.066480000000000011307; geometry collision mesh filename=./drive_palonier.stl; collision mesh filename=./passive_palonier.stl
- link hip_roll_assembly_2: mass 0.06648000000000005294 -> 0.066480000000000011307; geometry collision mesh filename=./drive_palonier.stl; collision mesh filename=./passive_palonier.stl
- link knee_and_ankle_assembly: geometry collision mesh filename=./drive_palonier.stl; collision mesh filename=./left_cache.stl
- link knee_and_ankle_assembly_2: mass 0.072590000000000057256 -> 0.072590000000000015623; geometry collision mesh filename=./drive_palonier.stl; collision mesh filename=./left_knee_to_ankle_left_sheet.stl
- link knee_and_ankle_assembly_3: mass 0.12407000000000001361 -> 0.12407000000000004136; geometry collision mesh filename=./drive_palonier.stl; collision mesh filename=./left_knee_to_ankle_left_sheet.stl
- link knee_and_ankle_assembly_4: mass 0.072590000000000057256 -> 0.072590000000000015623; geometry collision mesh filename=./drive_palonier.stl; collision mesh filename=./left_knee_to_ankle_left_sheet.stl
- link left_antenna_holder: mass 0.0042162890957708797426 -> 0.00421628909577088061
- link left_roll_to_pitch_assembly: mass 0.075160000000000060094 -> 0.075160000000000004583; geometry collision mesh filename=./drive_palonier.stl; collision mesh filename=./left_roll_to_pitch.stl
- link neck_pitch_assembly: mass 0.066180000000000058225 -> 0.066180000000000016591; geometry collision mesh filename=./drive_palonier.stl; collision mesh filename=./neck_left_sheet.stl
- link neck_yaw_assembly: mass 0.09180988857925044544 -> 0.091809888579250376051; geometry collision mesh filename=./drive_palonier.stl; collision mesh filename=./head_yaw_to_roll.stl
- link right_antenna_holder: mass 0.004216286984950681424 -> 0.0042162869849506796893
- link right_roll_to_pitch_assembly: mass 0.075160000000000060094 -> 0.075160000000000004583; geometry collision mesh filename=./drive_palonier.stl; collision mesh filename=./passive_palonier.stl
- link trunk_assembly: geometry collision mesh filename=./battery_pack_lid.stl; collision mesh filename=./bms.stl
Joints:
- joint head_frame: origin xyz=0.04245000000000057061 7.4178402136026999614e-16 0.035949999999999988909 rpy=2.2204460492701854731e-16 1.570796326794896336 0 -> xyz=0.04244999999999957141 2.135878279796443735e-17 0.035950000000000377487 rpy=-0 1.570796326794896558 0
- joint head_pitch: limit lower=-0.785398163397448279 upper=0.785398163397448279 effort=20 velocity=200 -> lower=-0.785398163397448279 upper=0.785398163397448279 effort=1 velocity=20; origin xyz=8.6736173798840354721e-19 0.066000000000000016986 -3.4694469519536141888e-18 rpy=-1.4406834481465239151e-16 -1.1423136877781657605e-16 1.1213426021061680001e-13 -> xyz=-5.42101086242752217e-17 0.066000000000000086375 -1.0408340855860842566e-17 rpy=-1.9479487599482720301e-16 -1.1423136863502905442e-16 1.7347234747146296461e-18
- joint head_roll: limit lower=-0.52359877559829881566 upper=0.52359877559829881566 effort=20 velocity=200 -> lower=-0.52359877559829881566 upper=0.52359877559829881566 effort=1 velocity=20; origin xyz=0.040950000000000097433 -1.7527483370943786056e-16 -0.019149999999999778311 rpy=-7.3227915058204641542e-14 -1.570796326794896336 0 -> xyz=0.040950000000000000289 -4.2214766838438722019e-16 -0.019149999999999833822 rpy=1.2411687278497551329e-14 -1.5707963267948830133 0
- joint head_yaw: limit lower=-2.7925268031909271649 upper=2.7925268031909271649 effort=20 velocity=200 -> lower=-2.7925268031909271649 upper=2.7925268031909271649 effort=1 velocity=20; origin xyz=-1.6913553890773869171e-17 0.056999999999999939604 0.019050000000000014838 rpy=-1.570796326794896558 7.3522809646371816617e-14 6.1232339957365034931e-17 -> xyz=-9.9746599868666407929e-18 0.056999999999999967359 0.019050000000000014838 rpy=-1.570796326794896558 -1.3706437208012195828e-25 6.1232339958582419871e-17
- joint left_ankle: limit lower=-1.570796326794896558 upper=1.570796326794896558 effort=20 velocity=200 -> lower=-1.570796326794896558 upper=1.570796326794896558 effort=1 velocity=20; origin xyz=-3.4694469519536141888e-17 -0.078650000000000178102 9.99999999999751088e-05 rpy=-2.6413756774523519415e-16 1.2220841311108591179e-26 2.7755576181993178136e-17 -> xyz=-7.9103390504542403505e-16 -0.078649999999999428701 9.9999999999794697558e-05 rpy=1.636340693842024721e-16 1.1379785959205303308e-15 -2.7755597583208935156e-17
- joint left_antenna: limit lower=-1.570796326794896558 upper=1.570796326794896558 effort=20 velocity=200 -> lower=-1.570796326794896558 upper=1.570796326794896558 effort=1 velocity=20; origin xyz=0.00070406945503534434927 0.060662837687359784378 0.11643485329544212004 rpy=-3.1415926535896234739 1.3045791727887248168 1.3234423712232488146 -> xyz=0.00070406945503187490232 0.060662837687359048855 0.1164348532954449511 rpy=-3.1415926535897802374 1.3045791727887245948 1.3234423712230847237
- joint left_foot_frame: origin xyz=0.00049999999999996574962 -0.036224999999999729638 0.01955000000000034488 rpy=-1.570796326794896558 4.8789097742003279458e-18 8.5828066488045564267e-28 -> xyz=0.00049999999999995187183 -0.036224999999999729638 0.019550000000000331002 rpy=-1.570796326794896558 4.8789097652664912905e-18 2.353432088828639061e-23
- joint left_hip_pitch: limit lower=-1.570796326794896558 upper=0.72359877559829881566 effort=20 velocity=200 -> lower=-1.2217304763960306069 upper=0.52359877559829881566 effort=1 velocity=20; origin xyz=0.074149999999999799405 1.3959102970750869588e-18 0.035109999999999912113 rpy=3.141592653589793116 1.5707963267948952257 0 -> xyz=0.074149999999999799405 -1.9529191631895148618e-17 0.035109999999999898235 rpy=3.141592653589793116 1.570796326794896336 0
- joint left_hip_roll: limit lower=-0.43633231299858238339 upper=0.43633231299858238339 effort=20 velocity=200 -> lower=-0.43633231299858238339 upper=0.43633231299858238339 effort=1 velocity=20; origin xyz=0.019050000000003241424 2.0469737016526323714e-15 -0.046015000000000895464 rpy=-1.5707963267949442976 1.0251581517556108667e-13 1.5707963267946023489 -> xyz=0.019050000000003588368 4.3576253716537394212e-15 -0.046015000000001519964 rpy=-1.5707963267949396347 9.7936145200150713608e-14 1.5707963267946445374
- joint left_hip_yaw: limit lower=-0.52359877559829881566 upper=0.52359877559829881566 effort=20 velocity=200 -> lower=-0.52359877559829881566 upper=0.52359877559829881566 effort=1 velocity=20; origin xyz=-0.019000000000000290962 0.035000000000001273148 0.045940938812378845357 rpy=-2.0757017677015319346e-16 -2.1982415887547258194e-14 -7.6136910267405882653e-27 -> xyz=-0.018999999999998434808 0.035000000000000974776 0.04594093881237738819 rpy=-1.5205902553582758499e-16 -2.2037927038784495587e-14 -6.3658912806794774433e-27
- joint left_knee: limit lower=-1.570796326794896558 upper=1.570796326794896558 effort=20 velocity=200 -> lower=-1.570796326794896558 upper=1.570796326794896558 effort=1 velocity=20; origin xyz=1.3877787807814456755e-17 -0.078650000000000011569 9.9999999999961231012e-05 rpy=-2.6413756781799972404e-16 -2.7339812777890022088e-26 0 -> xyz=-2.9837243786801082024e-16 -0.078650000000000871991 9.99999999999751088e-05 rpy=-2.6413758326899544516e-16 -7.0075679691128679348e-24 -2.4877517507049828295e-26
- joint neck_pitch: limit lower=-0.34906585039886589561 upper=1.1344640137963142301 effort=20 velocity=200 -> lower=-0.34906585039886589561 upper=1.1344640137963142301 effort=1 velocity=20; origin xyz=0.00099999999999896352354 0.019150000000000326483 0.090000938812376238274 rpy=1.570796326794896558 8.9928064994637667153e-14 6.1232449686014378908e-17 -> xyz=0.00099999999999899474856 0.019150000000000326483 0.090000938812376224396 rpy=1.57079632679489678 -2.2204460492503130808e-14 6.1232449680326617825e-17
- joint right_ankle: limit lower=-1.570796326794896558 upper=1.570796326794896558 effort=20 velocity=200 -> lower=-1.570796326794896558 upper=1.570796326794896558 effort=1 velocity=20; origin xyz=-6.9388939039072283776e-18 -0.078650000000000039324 9.9999999999961231012e-05 rpy=-2.6413756984180028828e-16 -6.9382288127881716121e-25 -5.1722034616178551878e-17 -> xyz=1.3877787807814456755e-17 -0.078649999999999928302 0.00010000000000004449774 rpy=-2.6413812280837946538e-16 -1.7764738567684265366e-22 4.6805027693161558698e-25
- joint right_antenna: limit lower=-1.570796326794896558 upper=1.570796326794896558 effort=20 velocity=200 -> lower=-1.570796326794896558 upper=1.570796326794896558 effort=1 velocity=20; origin xyz=0.00070406945503534434927 -0.06066283768735826476 0.11643485329544212004 rpy=3.1415926535896230298 1.3045791727887245948 -1.3234423712232490367 -> xyz=0.00070406945503675988363 -0.060662837687358986405 0.11643485329544003837 rpy=-3.1415926535897802374 1.3045791727887252609 -1.3234423712230598547
- joint right_foot_frame: origin xyz=0.0005000000000002155498 -0.036224999999999840661 0.019550000000000664069 rpy=-1.570796326794896558 9.1691846176123393012e-16 1.3322725304659061714e-15 -> xyz=0.00050000000000022942759 -0.036224999999999812905 0.019550000000000553046 rpy=-1.570796326794896558 -2.2055201956572090666e-25 -2.8950564132886956449e-25
- joint right_hip_pitch: limit lower=-0.72359877559829881566 upper=1.5707304763960306069 effort=20 velocity=200 -> lower=-0.52359877559829881566 upper=1.2217304763960306069 effort=1 velocity=20; origin xyz=-0.074149999999999799405 3.1868767607495795957e-16 0.035110000000000016196 rpy=-2.3836094894413110414e-24 1.570796326794896336 0 -> xyz=-0.074149999999999771649 5.1732706660145844069e-16 0.035110000000000037013 rpy=-6.1899281068357555747e-22 1.570796326794896336 0
- joint right_hip_roll: limit lower=-0.43633231299858238339 upper=0.43633231299858238339 effort=20 velocity=200 -> lower=-0.43633231299858238339 upper=0.43633231299858238339 effort=1 velocity=20; origin xyz=0.019050000000008261714 3.78516662458139308e-14 -0.046015000000003032643 rpy=-1.5707963267947879782 -8.4491074221037422062e-14 1.5707963267945974639 -> xyz=0.019050000000008570494 4.0564773762241657096e-14 -0.046015000000004170622 rpy=-1.5707963267947786523 -8.9077711856609251111e-14 1.5707963267946440933
- joint right_hip_yaw: limit lower=-0.52359877559829881566 upper=0.52359877559829881566 effort=20 velocity=200 -> lower=-0.52359877559829881566 upper=0.52359877559829881566 effort=1 velocity=20; origin xyz=-0.018999999999998431338 -0.03500000000000151601 0.045940938812377415945 rpy=-4.6224992538811313716e-16 -2.2037927038832600325e-14 -1.6653345370219725828e-16 -> xyz=-0.018999999999998431338 -0.03500000000000151601 0.045940938812377415945 rpy=-5.7327222785292536251e-16 -2.1926904736366604217e-14 -2.7755575616618406396e-16
- joint right_knee: limit lower=-1.570796326794896558 upper=1.570796326794896558 effort=20 velocity=200 -> lower=-1.570796326794896558 upper=1.570796326794896558 effort=1 velocity=20; origin xyz=-6.9388939039072283776e-18 0.078649999999999414824 0.036999999999999658162 rpy=3.141592653589793116 -2.0819102970830263503e-24 5.0289882707839502595e-30 -> xyz=1.3877787807814456755e-17 0.078649999999999137268 0.036999999999999574896 rpy=3.141592653589793116 -5.3297228769912622595e-22 -2.2267995332275346432e-26

Commit message: simplify urdf

File: awd/data/assets/mini2_bdx/mini2_bdx.urdf (robot description, URDF)
Before this commit: robot onshape, 21 links, 20 joints
Links:
- link head_assembly: geometry collision mesh filename=./head.stl; collision mesh filename=./head_bot_sheet.stl
- link hip_roll_assembly: geometry collision mesh filename=./roll_motor_bottom.stl; collision mesh filename=./roll_motor_top.stl
- link hip_roll_assembly_2: geometry collision mesh filename=./roll_motor_bottom.stl; collision mesh filename=./roll_motor_top.stl
- link knee_and_ankle_assembly: geometry collision mesh filename=./left_cache.stl; collision mesh filename=./left_knee_to_ankle_left_sheet.stl
- link knee_and_ankle_assembly_2: geometry collision mesh filename=./left_knee_to_ankle_left_sheet.stl; collision mesh filename=./left_knee_to_ankle_right_sheet.stl
- link knee_and_ankle_assembly_3: geometry collision mesh filename=./left_knee_to_ankle_left_sheet.stl; collision mesh filename=./left_knee_to_ankle_right_sheet.stl
- link knee_and_ankle_assembly_4: geometry collision mesh filename=./left_knee_to_ankle_left_sheet.stl; collision mesh filename=./left_knee_to_ankle_right_sheet.stl
- link left_roll_to_pitch_assembly: geometry collision mesh filename=./left_roll_to_pitch.stl; visual mesh filename=./left_roll_to_pitch.stl
- link neck_pitch_assembly: geometry collision mesh filename=./neck_left_sheet.stl; collision mesh filename=./neck_right_sheet.stl
- link neck_yaw_assembly: geometry collision mesh filename=./head_yaw_to_roll.stl; visual mesh filename=./head_yaw_to_roll.stl
- link right_roll_to_pitch_assembly: geometry collision mesh filename=./right_roll_to_pitch.stl; visual mesh filename=./right_roll_to_pitch.stl
- link trunk_assembly: geometry collision mesh filename=./body_back.stl; collision mesh filename=./body_front.stl
